File: blocks/blocks.sch (KiCad schematic (older format))
At the start: 28 parts, among them IC1 ATTINY85-S, P1 PAD_R, P2 PAD_L, P3 PAD_RX, P4 PAD_TX, P5 ISP, SW1 SW_PUSH

Commit message: Fixed wrong pull up reference for RESET input
Connections:
- net +3V3: now also R5.1
- net VCC: no longer R5.1
Other:
- moved on the sheet: R5
Changed lines of the file:
@@
 L R R5
 U 1 1 571CFCA4
-P 5000 4300
-F 0 "R5" V 5080 4300 50  0000 C CNN
-F 1 "1k" V 5000 4300 50  0000 C CNN
-F 2 "Resistors_SMD:R_0805_HandSoldering" V 4930 4300 50  0001 C CNN
-F 3 "" H 5000 4300 50  0000 C CNN
-	1    5000 4300
+P 4800 4300
+F 0 "R5" V 4880 4300 50  0000 C CNN
+F 1 "1k" V 4800 4300 50  0000 C CNN
+F 2 "Resistors_SMD:R_0805_HandSoldering" V 4730 4300 50  0001 C CNN
+F 3 "" H 4800 4300 50  0000 C CNN
+	1    4800 4300
 	0    1    -1   0
 $EndComp
 Wire Wire Line
-	5150 4300 5400 4300
-Connection ~ 5400 4300
-Wire Wire Line
-	4850 4300 4250 4300
+	4650 4300 4250 4300
 Wire Wire Line
 	4250 4300 4250 4750
@@
 Wire Wire Line
 	7100 1100 7000 1100
+$Comp
+L +3.3V #PWR017
+U 1 1 571DD32E
+P 5150 4200
+F 0 "#PWR017" H 5150 4050 50  0001 C CNN
+F 1 "+3.3V" H 5150 4340 50  0000 C CNN
+F 2 "" H 5150 4200 50  0000 C CNN
+F 3 "" H 5150 4200 50  0000 C CNN
+	1    5150 4200
+	1    0    0    -1
+$EndComp
+Wire Wire Line
+	4950 4300 5150 4300
+Wire Wire Line
+	5150 4300 5150 4200
 $EndSCHEMATC

Commit message: Added mounting holes and changed Zener diode on brick pcb
Parts:
- removed D1: BAR43S, TO_SOT_Packages_SMD:SOT-23_Handsoldering, symbol D_Schottky_x2_Serial_AKC
- removed D2: 3V3, Diodes_SMD:MELF_Handsoldering, symbol ZENER
- added D1: 3V3, TO_SOT_Packages_SMD:SOT-23, symbol BZX84C
Connections:
- net +3V3: now also R1.1, D1.3 (K)
- net GND: now also D1.1 (A)
Other:
- moved on the sheet: P1, P2, R1
Changed lines of the file:
@@
-$EndComp
-$Comp
-L ZENER D2
-U 1 1 571CCC6B
-P 2550 1450
-F 0 "D2" H 2550 1550 50  0000 C CNN
-F 1 "3V3" H 2550 1350 50  0000 C CNN
-F 2 "Diodes_SMD:MELF_Handsoldering" H 2550 1450 50  0001 C CNN
-F 3 "" H 2550 1450 50  0000 C CNN
-	1    2550 1450
-	0    1    1    0
 $EndComp
 $Comp
 L R R1
 U 1 1 571CCCD9
-P 1450 1150
-F 0 "R1" V 1530 1150 50  0000 C CNN
-F 1 "100R" V 1450 1150 50  0000 C CNN
-F 2 "Resistors_SMD:R_0805_HandSoldering" V 1380 1150 50  0001 C CNN
-F 3 "" H 1450 1150 50  0000 C CNN
-	1    1450 1150
+P 2050 1150
+F 0 "R1" V 2130 1150 50  0000 C CNN
+F 1 "100R" V 2050 1150 50  0000 C CNN
+F 2 "Resistors_SMD:R_0805_HandSoldering" V 1980 1150 50  0001 C CNN
+F 3 "" H 2050 1150 50  0000 C CNN
+	1    2050 1150
 	0    1    1    0
 $EndComp
@@
 	2550 1050 2550 1250
 Wire Wire Line
-	2400 1150 2850 1150
+	2200 1150 2850 1150
 Connection ~ 2550 1150
 $Comp
@@
 L CONN_01X01 P1
 U 1 1 571CCF17
-P 900 1150
-F 0 "P1" H 900 1250 50  0000 C CNN
-F 1 "PAD_R" V 1000 1150 50  0000 C CNN
-F 2 "custom:BigPad" H 900 1150 50  0001 C CNN
-F 3 "" H 900 1150 50  0000 C CNN
-	1    900  1150
+P 1500 1150
+F 0 "P1" H 1500 1250 50  0000 C CNN
+F 1 "PAD_R" V 1600 1150 50  0000 C CNN
+F 2 "custom:BigPad" H 1500 1150 50  0001 C CNN
+F 3 "" H 1500 1150 50  0000 C CNN
+	1    1500 1150
 	-1   0    0    1
 $EndComp
@@
 L CONN_01X01 P2
 U 1 1 571CCFAC
-P 900 1750
-F 0 "P2" H 900 1850 50  0000 C CNN
-F 1 "PAD_L" V 1000 1750 50  0000 C CNN
-F 2 "custom:HugePad" H 900 1750 50  0001 C CNN
-F 3 "" H 900 1750 50  0000 C CNN
-	1    900  1750
-	-1   0    0    1
-$EndComp
-Wire Wire Line
-	1100 1750 2850 1750
+P 1500 1750
+F 0 "P2" H 1500 1850 50  0000 C CNN
+F 1 "PAD_L" V 1600 1750 50  0000 C CNN
+F 2 "custom:HugePad" H 1500 1750 50  0001 C CNN
+F 3 "" H 1500 1750 50  0000 C CNN
+	1    1500 1750
+	-1   0    0    1
+$EndComp
+Wire Wire Line
+	1700 1750 2850 1750
 Connection ~ 2550 1750
 Wire Wire Line
-	1100 1150 1300 1150
+	1700 1150 1900 1150
 $Comp
 L CONN_01X01 P3
@@
 L VCC #PWR014
 U 1 1 571CF429
-P 1200 1050
-F 0 "#PWR014" H 1200 900 50  0001 C CNN
-F 1 "VCC" H 1200 1200 50  0000 C CNN
-F 2 "" H 1200 1050 50  0000 C CNN
-F 3 "" H 1200 1050 50  0000 C CNN
-	1    1200 1050
-	1    0    0    -1
-$EndComp
-Wire Wire Line
-	1200 1050 1200 1150
-Connection ~ 1200 1150
+P 1800 1050
+F 0 "#PWR014" H 1800 900 50  0001 C CNN
+F 1 "VCC" H 1800 1200 50  0000 C CNN
+F 2 "" H 1800 1050 50  0000 C CNN
+F 3 "" H 1800 1050 50  0000 C CNN
+	1    1800 1050
+	1    0    0    -1
+$EndComp
+Wire Wire Line
+	1800 1050 1800 1150
+Connection ~ 1800 1150
 $Comp
 L VCC #PWR015
@@
 	8400 3450 8400 3750
 Connection ~ 8400 3750
-$Comp
-L D_Schottky_x2_Serial_AKC D1
-U 1 1 571CDF2B
-P 2100 1150
-F 0 "D1" H 2150 1050 50  0000 C CNN
-F 1 "BAR43S" H 2100 1250 50  0000 C CNN
-F 2 "TO_SOT_Packages_SMD:SOT-23_Handsoldering" H 2100 1150 50  0001 C CNN
-F 3 "" H 2100 1150 50  0000 C CNN
-	1    2100 1150
-	1    0    0    1
-$EndComp
-Wire Wire Line
-	1600 1150 1800 1150
-Wire Wire Line
-	1700 850  1700 1150
-Connection ~ 1700 1150
-Wire Wire Line
-	2100 950  2100 850
-Wire Wire Line
-	2100 850  1700 850
 Text Label 6200 3200 0    60   ~ 0
 LED2
@@
 Wire Wire Line
 	5150 4300 5150 4200
+$Comp
+L BZX84C D1
+U 1 1 574C2955
+P 2550 1450
+F 0 "D1" H 2550 1550 50  0000 C CNN
+F 1 "3V3" H 2550 1350 50  0000 C CNN
+F 2 "TO_SOT_Packages_SMD:SOT-23" H 2550 1450 50  0001 C CNN
+F 3 "" H 2550 1450 50  0000 C CNN
+	1    2550 1450
+	0    1    1    0
+$EndComp
 $EndSCHEMATC
