File: remote/remote.sch (KiCad schematic (older format))
At the start: 40 parts, among them IC1 ATMEGA328P-A, P1 CON_TX, P2 CON_TX, P3 BRICK_P, P4 BRICK_N, P5 HD44780_LCD, P6 CONN_02X03, Q1 BC349, Q2 BC349, Q3 BC358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

Commit message: finished layouting the collector unit
Parts:
- added CON1: BARREL_JACK, Connect:BARREL_JACK, symbol BARREL_JACK
- added JP1: JUMPER, Resistors_SMD:R_0805_HandSoldering, symbol JUMPER
- added P7: BRICK_P, custom:SmallFoilCon, symbol CONN_01X01
- added P8: BRICK_N, custom:BigFoilCon, symbol CONN_01X01
- C2, C3, C4, C5: value CP -> 1u; footprint (none) -> Capacitors_Tantalum_SMD:TantalC_SizeA_EIA-3216_HandSoldering
- P1, P3: footprint (none) -> custom:SmallFoilCon
- P2: value CON_TX -> CON_RX; footprint (none) -> custom:SmallFoilCon
- P4: footprint (none) -> custom:BigFoilCon
- RV1: footprint (none) -> custom:Cermet_Model23
- SW1: footprint (none) -> custom:Schurter_LSG_1301
- U1, U2: value 78L03 -> TS2940 CP33; footprint (none) -> TO_SOT_Packages_SMD:TO-252-2Lead
- U3: footprint (none) -> custom:RFM75
- Y1: footprint (none) -> Crystals:Crystal_HC49-U_Vertical
Connections:
- net +3V3: now also JP1.1
- net +5V: now also JP1.2
- net +BATT: now also CON1.1
- net GND: now also CON1.2, CON1.3, P8.1 (P1)
- net at C5.1, P3.1 (P1), U2.VO: now also P7.1 (P1)
Changed lines of the file:
@@
 F 0 "Y1" H 9850 3000 50  0000 C CNN
 F 1 "12MHz" H 9850 2700 50  0000 C CNN
-F 2 "" H 9850 2850 50  0001 C CNN
+F 2 "Crystals:Crystal_HC49-U_Vertical" H 9850 2850 50  0001 C CNN
 F 3 "" H 9850 2850 50  0000 C CNN
 	1    9850 2850
@@
 F 0 "P1" H 1250 6500 50  0000 C CNN
 F 1 "CON_TX" V 1350 6400 50  0000 C CNN
-F 2 "" H 1250 6400 50  0001 C CNN
+F 2 "custom:SmallFoilCon" H 1250 6400 50  0001 C CNN
 F 3 "" H 1250 6400 50  0000 C CNN
 	1    1250 6400
@@
 P 2700 6400
 F 0 "P2" H 2700 6500 50  0000 C CNN
-F 1 "CON_TX" V 2800 6400 50  0000 C CNN
-F 2 "" H 2700 6400 50  0001 C CNN
+F 1 "CON_RX" V 2800 6400 50  0000 C CNN
+F 2 "custom:SmallFoilCon" H 2700 6400 50  0001 C CNN
 F 3 "" H 2700 6400 50  0000 C CNN
 	1    2700 6400
@@
 P 3350 2450
 F 0 "U2" H 3500 2254 50  0000 C CNN
-F 1 "78L03" H 3350 2650 50  0000 C CNN
-F 2 "" H 3350 2450 50  0001 C CNN
+F 1 "TS2940 CP33" H 3350 2650 50  0000 C CNN
+F 2 "TO_SOT_Packages_SMD:TO-252-2Lead" H 3350 2450 50  0001 C CNN
 F 3 "" H 3350 2450 50  0000 C CNN
 	1    3350 2450
@@
 P 2800 2750
 F 0 "C3" H 2825 2850 50  0000 L CNN
-F 1 "CP" H 2825 2650 50  0000 L CNN
-F 2 "" H 2838 2600 50  0001 C CNN
+F 1 "1u" H 2825 2650 50  0000 L CNN
+F 2 "Capacitors_Tantalum_SMD:TantalC_SizeA_EIA-3216_HandSoldering" H 2838 2600 50  0001 C CNN
 F 3 "" H 2800 2750 50  0000 C CNN
 	1    2800 2750
@@
 P 3900 2750
 F 0 "C5" H 3925 2850 50  0000 L CNN
-F 1 "CP" H 3925 2650 50  0000 L CNN
-F 2 "" H 3938 2600 50  0001 C CNN
+F 1 "1u" H 3925 2650 50  0000 L CNN
+F 2 "Capacitors_Tantalum_SMD:TantalC_SizeA_EIA-3216_HandSoldering" H 3938 2600 50  0001 C CNN
 F 3 "" H 3900 2750 50  0000 C CNN
 	1    3900 2750
@@
 $EndComp
 Wire Wire Line
-	3900 3050 3900 2900
+	3900 2900 3900 3250
 Wire Wire Line
 	3750 2400 4050 2400
 Wire Wire Line
-	3900 2400 3900 2600
+	3900 2200 3900 2600
 $Comp
 L Q_PNP_BEC Q4
@@
 F 0 "P3" H 4250 2500 50  0000 C CNN
 F 1 "BRICK_P" H 4550 2400 50  0000 C CNN
-F 2 "" H 4250 2400 50  0001 C CNN
+F 2 "custom:SmallFoilCon" H 4250 2400 50  0001 C CNN
 F 3 "" H 4250 2400 50  0000 C CNN
 	1    4250 2400
@@
 F 0 "P4" H 4250 3150 50  0000 C CNN
 F 1 "BRICK_N" H 4550 3050 50  0000 C CNN
-F 2 "" H 4250 3050 50  0001 C CNN
+F 2 "custom:BigFoilCon" H 4250 3050 50  0001 C CNN
 F 3 "" H 4250 3050 50  0000 C CNN
 	1    4250 3050
@@
 F 0 "SW1" H 2100 4410 50  0000 C CNN
 F 1 "SEND" H 2200 4300 50  0000 C CNN
-F 2 "" H 1950 4300 50  0001 C CNN
+F 2 "custom:Schurter_LSG_1301" H 1950 4300 50  0001 C CNN
 F 3 "" H 1950 4300 50  0000 C CNN
 	1    1950 4300
@@
 P 3200 4400
 F 0 "U1" H 3350 4204 50  0000 C CNN
-F 1 "78L03" H 3200 4600 50  0000 C CNN
-F 2 "" H 3200 4400 50  0001 C CNN
+F 1 "TS2940 CP33" H 3200 4600 50  0000 C CNN
+F 2 "TO_SOT_Packages_SMD:TO-252-2Lead" H 3200 4400 50  0001 C CNN
 F 3 "" H 3200 4400 50  0000 C CNN
 	1    3200 4400
@@
 P 2650 4700
 F 0 "C2" H 2675 4800 50  0000 L CNN
-F 1 "CP" H 2675 4600 50  0000 L CNN
-F 2 "" H 2688 4550 50  0001 C CNN
+F 1 "1u" H 2675 4600 50  0000 L CNN
+F 2 "Capacitors_Tantalum_SMD:TantalC_SizeA_EIA-3216_HandSoldering" H 2688 4550 50  0001 C CNN
 F 3 "" H 2650 4700 50  0000 C CNN
 	1    2650 4700
@@
 P 3750 4700
 F 0 "C4" H 3775 4800 50  0000 L CNN
-F 1 "CP" H 3775 4600 50  0000 L CNN
-F 2 "" H 3788 4550 50  0001 C CNN
+F 1 "1u" H 3775 4600 50  0000 L CNN
+F 2 "Capacitors_Tantalum_SMD:TantalC_SizeA_EIA-3216_HandSoldering" H 3788 4550 50  0001 C CNN
 F 3 "" H 3750 4700 50  0000 C CNN
 	1    3750 4700
@@
 F 0 "RV1" H 5350 5670 50  0000 C CNN
 F 1 "POT" H 5350 5750 50  0000 C CNN
-F 2 "" H 5350 5750 50  0001 C CNN
+F 2 "custom:Cermet_Model23" H 5350 5750 50  0001 C CNN
 F 3 "" H 5350 5750 50  0000 C CNN
 	1    5350 5750
@@
 Connection ~ 5700 5750
 Wire Wire Line
-	5200 5750 5050 5750
+	4950 5750 5200 5750
 Connection ~ 5050 5750
 Wire Wire Line
@@
 F 0 "U3" H 9250 6000 60  0000 C CNN
 F 1 "RFM75" H 9700 5650 60  0000 C CNN
-F 2 "" H 9600 5650 60  0001 C CNN
+F 2 "custom:RFM75" H 9600 5650 60  0001 C CNN
 F 3 "" H 9600 5650 60  0000 C CNN
 	1    9600 5650
@@
 Wire Wire Line
 	9350 950  9200 950
+$Comp
+L BARREL_JACK CON1
+U 1 1 574D972F
+P 5350 1150
+F 0 "CON1" H 5350 1400 50  0000 C CNN
+F 1 "BARREL_JACK" H 5350 950 50  0000 C CNN
+F 2 "Connect:BARREL_JACK" H 5350 1150 50  0001 C CNN
+F 3 "" H 5350 1150 50  0000 C CNN
+	1    5350 1150
+	-1   0    0    -1
+$EndComp
+$Comp
+L +BATT #PWR026
+U 1 1 574D981B
+P 4900 1000
+F 0 "#PWR026" H 4900 850 50  0001 C CNN
+F 1 "+BATT" H 4900 1140 50  0000 C CNN
+F 2 "" H 4900 1000 50  0000 C CNN
+F 3 "" H 4900 1000 50  0000 C CNN
+	1    4900 1000
+	1    0    0    -1
+$EndComp
+Wire Wire Line
+	4700 1000 4700 1250
+Wire Wire Line
+	4700 1250 5050 1250
+$Comp
+L GND #PWR027
+U 1 1 574D9AA2
+P 4700 1000
+F 0 "#PWR027" H 4700 750 50  0001 C CNN
+F 1 "GND" H 4700 850 50  0000 C CNN
+F 2 "" H 4700 1000 50  0000 C CNN
+F 3 "" H 4700 1000 50  0000 C CNN
+	1    4700 1000
+	-1   0    0    1
+$EndComp
+Wire Wire Line
+	5050 1150 4900 1150
+Wire Wire Line
+	4900 1150 4900 1250
+Connection ~ 4900 1250
+Wire Wire Line
+	4900 1000 4900 1050
+Wire Wire Line
+	4900 1050 5050 1050
+$Comp
+L CONN_01X01 P7
+U 1 1 574DC2CF
+P 4250 2200
+F 0 "P7" H 4250 2300 50  0000 C CNN
+F 1 "BRICK_P" H 4550 2200 50  0000 C CNN
+F 2 "custom:SmallFoilCon" H 4250 2200 50  0001 C CNN
+F 3 "" H 4250 2200 50  0000 C CNN
+	1    4250 2200
+	1    0    0    -1
+$EndComp
+$Comp
+L CONN_01X01 P8
+U 1 1 574DC367
+P 4250 3250
+F 0 "P8" H 4250 3350 50  0000 C CNN
+F 1 "BRICK_N" H 4550 3250 50  0000 C CNN
+F 2 "custom:BigFoilCon" H 4250 3250 50  0001 C CNN
+F 3 "" H 4250 3250 50  0000 C CNN
+	1    4250 3250
+	1    0    0    -1
+$EndComp
+Wire Wire Line
+	3900 3250 4050 3250
+Wire Wire Line
+	4050 2200 3900 2200
+$Comp
+L +3.3V #PWR028
+U 1 1 574DB2AF
+P 4250 5650
+F 0 "#PWR028" H 4250 5500 50  0001 C CNN
+F 1 "+3.3V" H 4250 5790 50  0000 C CNN
+F 2 "" H 4250 5650 50  0000 C CNN
+F 3 "" H 4250 5650 50  0000 C CNN
+	1    4250 5650
+	1    0    0    -1
+$EndComp
+$Comp
+L JUMPER JP1
+U 1 1 574DB312
+P 4650 5750
+F 0 "JP1" H 4650 5900 50  0000 C CNN
+F 1 "JUMPER" H 4650 5670 50  0000 C CNN
+F 2 "Resistors_SMD:R_0805_HandSoldering" H 4650 5750 50  0001 C CNN
+F 3 "" H 4650 5750 50  0000 C CNN
+	1    4650 5750
+	1    0    0    -1
+$EndComp
+Wire Wire Line
+	4250 5650 4250 5750
+Wire Wire Line
+	4250 5750 4350 5750
 $EndSCHEMATC
